File: pcb/exixe19a/exixe19a.kicad_sch (KiCad schematic)
At the start: 39 parts, among them J1 Conn_01x07, J2 Conn_01x07, Q1 BF820W, Q10 BF820W, Q11 BF820W, Q3 MSB92W, Q4 BF820W, Q5 BF820W, Q6 BF820W, Q7 BF820W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

Commit message: pcb design for IN-19 tubes
Parts:
- D1: footprint LED_SMD:LED_Avago_PLCC4_3.2x2.8mm_CW -> LED_SMD:LED_RGB_Wuerth-PLCC4_3.2x2.8mm_150141M173100
Changed lines of the file:
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@@
 			)
 		)
-		(property "Footprint" "LED_SMD:LED_Avago_PLCC4_3.2x2.8mm_CW"
+		(property "Footprint" "LED_SMD:LED_RGB_Wuerth-PLCC4_3.2x2.8mm_150141M173100"
 			(at 31.75 30.48 0)
 			(effects
@@
 			)
 		)
-		(property "Description" "RGB LED, anode/blue/red/green"
+		(property "Description" "Wurth Elektronik2 V, 3.2 V RGB LED 3528 (1411) SMD, WL-SFTW 150141M173100"
 			(at 31.75 31.75 0)
 			(effects
